File: Audio_Amplifier d class.kicad_sch (KiCad schematic)
At the start: 3 parts, among them U1 TL494, U2 IR2110, U3 NE555D

Commit message: Add full Class-D amplifier schematic from reference design.
Co-authored-by: Cursor <cursoragent@cursor.com>
Parts:
- removed U1: TL494, Package_SO:SOIC-8_3.9x4.9mm_P1.27mm, symbol Regulator_Controller:TL494
- removed U2: IR2110, Package_DIP:DIP-14_W7.62mm, symbol Driver_FET:IR2110
- removed U3: NE555D, Package_SO:SOIC-8_3.9x4.9mm_P1.27mm, symbol Timer:NE555D
- added C1, C3, C4, C5, C7, C8, C9: 100n, symbol Device:C
- added C10, C11: 470n, symbol Device:C
- added C12: 10n, Capacitor_SMD:C_0201_0603Metric_Pad0.64x0.40mm_HandSolder, symbol Device:C
- added C13: 56p, symbol Device:C
- added C14: 100u, Capacitor_SMD:C_1206_3216Metric_Pad1.33x1.80mm_HandSolder, symbol Device:C
- added C15: 100n, Capacitor_SMD:C_0603_1608Metric_Pad1.08x0.95mm_HandSolder, symbol Device:C
- added C16, C17: 47u, symbol Device:C_Polarized
- added C18: 1u, symbol Device:C
- added C19: 100n, Capacitor_SMD:C_0201_0603Metric_Pad0.64x0.40mm_HandSolder, symbol Device:C
- added C2, C6: 10u, symbol Device:C_Polarized
- added C20: 56p, Capacitor_SMD:C_0201_0603Metric_Pad0.64x0.40mm_HandSolder, symbol Device:C
- added C21: 1n, symbol Device:C
- added C22: 10n, symbol Device:C
- added C23: 1u, symbol Device:C_Polarized
- added HL1: LED, symbol Device:LED
- added IC1, IC2: IR2110, symbol Driver_FET:IR2110
- added IC3: TL494, symbol Regulator_Controller:TL494
- added IC4: NE555D, symbol Timer:NE555D
- added J1: Вход, symbol Connector:Conn_01x02_Pin
- added J2: Вых1, symbol Connector:Conn_01x02_Pin
- added J3: Вых2, symbol Connector:Conn_01x02_Pin
- added L1, L2: 40uH, symbol Device:L
- added R1, R2, R3, R4: 24, symbol Device:R
- added R10, R23: 510, Resistor_SMD:R_0603_1608Metric_Pad0.98x0.95mm_HandSolder, symbol Device:R
- added R11, R12: 3k, symbol Device:R
- added R13, R14: 300, symbol Device:R
- added R15: 11k, symbol Device:R
- added R16, R22, R5, R6: 10k, symbol Device:R
- added R17: 1.5k, symbol Device:R_Potentiometer
- added R18: 0.05, symbol Device:R
- added R19: 1k, symbol Device:R_Potentiometer
- added R20: 1k, symbol Device:R
- added R21: 1M, symbol Device:R
- added R24: 47k, Resistor_SMD:R_0603_1608Metric_Pad0.98x0.95mm_HandSolder, symbol Device:R
- added R9: 1k, Resistor_SMD:R_0603_1608Metric_Pad0.98x0.95mm_HandSolder, symbol Device:R
- added VD1, VD4: SF16, symbol Device:D
- added VD2, VD3, VD5, VD6: 1N5219, symbol Device:D
- added VT1, VT2, VT3, VT4: IRFP460, symbol Transistor_FET:Q_NMOS_GDS
- added VT5: KT315, symbol Device:Q_NPN
Connections:
- new net: C5.1, C6.1, IC2.6 (VB), VD4.1 (K)
- new net: IC1.1 (LO), R2.1, VD3.1 (K)
- new net: C1.2, C2.2, IC1.5 (VS), L1.1, VT1.3 (S), VT2.2 (D)
- new net: C1.1, C2.1, IC1.6 (VB), VD1.1 (K)
- new net: IC1.7 (HO), R1.1, VD2.1 (K)
- new net: C19.2, C20.2, IC3.3 (FB)
- new net: R2.2, VD3.2 (A), VT2.1 (G)
- new net: R15.2, R17.1
- new net: IC2.1 (LO), R4.1, VD6.1 (K)
- new net: R4.2, VD6.2 (A), VT4.1 (G)
- new net: C23.1, IC4.6 (THRES), IC4.7 (DISCH), R21.2
- new net: C16.2, R11.1, R12.1
- new net: C21.1, R19.2, VT5.B
- new net: R1.2, VD2.2 (A), VT1.1 (G)
- new net: HL1.2 (A), R20.2
- new net: C13.2, R14.2
- new net: R3.2, VD5.2 (A), VT3.1 (G)
- new net: C19.1, R24.2
- new net: IC4.2 (TRIG), R22.2, VT5.C
- new net: IC2.7 (HO), R3.1, VD5.1 (K)
- new net: IC3.6 (RT), R9.1
- new net: C12.1, IC3.5 (CT)
- new net +12V: C14.1, C15.1, C22.1, C3.1, C4.2, C7.1, C8.1, IC1.3 (VCC), IC1.9 (VDD), IC2.3 (VCC), IC2.9 (VDD), IC3.12 (VCC), IC3.8 (C1), IC4.4 (~{RST}), IC4.5 (CONT), IC4.8 (VCC), R10.1, R15.1, R21.1, R22.1, VD1.2 (A), VD4.2 (A)
- new net +Upit: C9.1, VT1.2 (D), VT3.2 (D)
- new net AUDIO_IN: C18.1, J1.1 (Pin_1)
- new net C2: IC3.11 (C2), R10.2
- new net E1: IC3.9 (E1), R23.1
- new net GND: C10.2, C11.2, C12.2, C13.1, C14.2, C15.2, C16.1, C17.1, C17.2, C21.2, C22.2, C23.2, C3.2, C4.1, C5.2, C6.2, C7.2, C8.2, C9.2, HL1.1 (K), IC1.13 (VSS), IC1.2 (COM), IC2.13 (VSS), IC2.2 (COM), IC2.5 (VS), IC3.1 (1IN+), IC3.10 (E2), IC3.4 (DTC), IC3.7 (GND), IC4.1 (GND), J1.2 (Pin_2), J2.2 (Pin_2), J3.2 (Pin_2), L2.1, R11.2, R12.2, R14.1, R16.1, R16.2, R17.2, R17.3, R18.2, R19.3, R23.2, R5.2, R6.2, R9.2, VT3.3 (S), VT4.2 (D), VT5.E
- new net HIN: IC1.10 (HIN), IC2.10 (HIN)
- new net In2-: C20.1, IC3.15 (2IN-), R24.1
- new net LIN: IC1.12 (LIN), IC2.12 (LIN)
- new net OUT1: C10.1, J2.1 (Pin_1), L1.2, R5.1
- new net OUT2: C11.1, J3.1 (Pin_1), L2.2, R6.1
- new net SD: IC1.11 (SD), IC2.11 (SD), IC4.3 (OUT), R20.1
- new net SENSE: R18.1, R19.1, VT2.3 (S), VT4.3 (S)
- new net Uref: IC3.14 (REF), IC3.2 (1IN-)
Other:
- note added: "Вход"
- note added: "Вых1"
- note added: "Вых2"
- note added: "Перегрузка"
- note added: "Уст. 0"
- note added: "Уст. тока защиты"

Commit message: Revise the Class-D amplifier schematic and refresh used designators.
Co-authored-by: Cursor <cursoragent@cursor.com>
Parts:
- removed C16, C17: 47u, symbol Device:C_Polarized
- removed C18: 1u, symbol Device:C
- removed C23: 1u, symbol Device:C_Polarized
- removed C5, C7, C9: 100n, symbol Device:C
- removed C6: 10u, symbol Device:C_Polarized
- removed HL1: LED, symbol Device:LED
- removed J1: Вход, symbol Connector:Conn_01x02_Pin
- removed J2: Вых1, symbol Connector:Conn_01x02_Pin
- removed J3: Вых2, symbol Connector:Conn_01x02_Pin
- removed R11, R12: 3k, symbol Device:R
- removed R13, R14: 300, symbol Device:R
- removed R15: 11k, symbol Device:R
- removed R16: 10k, symbol Device:R
- removed R17: 1.5k, symbol Device:R_Potentiometer
- removed R20: 1k, symbol Device:R
- removed VD6: 1N5219, symbol Device:D
- added C16, C24, C28, C29, C30: 100n, Capacitor_SMD:C_0603_1608Metric_Pad1.08x0.95mm_HandSolder, symbol Device:C
- added C25: 1m, symbol Device:C
- added C26: 100n, Capacitor_SMD:C_0805_2012Metric_Pad1.18x1.45mm_HandSolder, symbol Device:C
- added C27: 47u, Capacitor_SMD:C_0805_2012Metric_Pad1.18x1.45mm_HandSolder, symbol Device:C
- added C9: 10u, symbol Device:C_Polarized
- added D1: LED, symbol Device:LED
- added R25, R26: 3k, Resistor_SMD:R_0603_1608Metric_Pad0.98x0.95mm_HandSolder, symbol Device:R
- added R27, R28: 300, Resistor_SMD:R_0603_1608Metric_Pad0.98x0.95mm_HandSolder, symbol Device:R
- added R29: 10k, Resistor_SMD:R_0603_1608Metric_Pad0.98x0.95mm_HandSolder, symbol Device:R
- added R30: 11k, Resistor_SMD:R_0603_1608Metric_Pad0.98x0.95mm_HandSolder, symbol Device:R
- added R31: 1k5, Resistor_SMD:R_0603_1608Metric_Pad0.98x0.95mm_HandSolder, symbol Device:R
- added R32: 1k, Capacitor_SMD:C_0603_1608Metric_Pad1.08x0.95mm_HandSolder, symbol Device:R
- added R33, R34: 10k, Capacitor_SMD:C_0603_1608Metric_Pad1.08x0.95mm_HandSolder, symbol Device:R
- added VD7: SF16, symbol Device:D
- C12, C19, C20: footprint Capacitor_SMD:C_0201_0603Metric_Pad0.64x0.40mm_HandSolder -> Capacitor_SMD:C_0603_1608Metric_Pad1.08x0.95mm_HandSolder
- C13: value 56p -> 100n; footprint (none) -> Capacitor_SMD:C_0603_1608Metric_Pad1.08x0.95mm_HandSolder
- C22: value 10n -> 100n; footprint (none) -> Capacitor_SMD:C_0603_1608Metric_Pad1.08x0.95mm_HandSolder
- VD4: value SF16 -> 1N5219
Connections:
- net +12V: now also C13.2, R22.2, VT5.C, C16.2, C29.2, R33.2, R34.1, VD7.2 (A); no longer C22.1, C3.1, IC4.5 (CONT), R22.1, VD4.2 (A)
- net C2: now also IC1.12 (LIN), IC2.10 (HIN)
- net E1: now also IC1.10 (HIN), IC2.12 (LIN)
- net GND: now also C22.1, R18.1, R19.2, C16.1, C26.2, C27.1, C29.1, C30.1, R27.1, R28.2; no longer C22.2, C3.2, IC2.5 (VS), L2.1, R18.2, VT3.3 (S), VT4.2 (D)
- net In2-: now also C24.1, C25.2, R26.2
- net SD: now also D1.2 (A), R33.1
- net Вход: now also C25.1
- net at IC2.6 (VB): now also C3.1, C9.1, VD7.1 (K); no longer VD4.1 (K)
- net IC1_LO: now reaches IC1.1 (LO), R2.1, VD3.1 (K)
- net IC1_VS: now reaches C1.2, C2.2, IC1.5 (VS), L1.1, VT1.3 (S), VT2.2 (D)
- net IC1_HO: now reaches IC1.7 (HO), R1.1, VD2.1 (K)
- net IC2_LO: now reaches IC2.1 (LO), R4.1
- net IC2_LO: now also VD5.1 (K)
- net at R4.2, VT4.1 (G): now also VD5.2 (A)
- net at IC4.6 (THRES), IC4.7 (DISCH), R21.2: now also C30.2
- net at C21.1, VT5.B: now also R19.1, R32.1; no longer R19.2
- net at R3.2, VT3.1 (G): now also VD4.2 (A); no longer VD5.2 (A)
- net IC2_HO: now reaches IC2.7 (HO), R3.1
- net IC2_HO: now also VD4.1 (K); no longer VD5.1 (K)
- net In2+: now reaches IC3.16 (2IN+)
- net In2+: now also C24.2, R25.2
- net +Upit renamed +Uпит
- removed net HIN: IC1.10 (HIN), IC2.10 (HIN)
- removed net LIN: IC1.12 (LIN), IC2.12 (LIN)
- net OUT1 renamed Out1
- net OUT2 renamed Out2
- net SENSE renamed Ток
- net Ток: now also R18.2, R32.2; no longer R18.1, R19.1
- new net: C27.2, C28.2, R25.1, R28.1, R30.2
- new net: C26.1, C28.1, R26.1, R27.2, R29.2
- new net: D1.1 (K), R34.2
- new net: IC4.2 (TRIG), R22.1
- new net: C22.2, IC4.5 (CONT)
- new net IC2_VS: C3.2, C9.2, IC2.5 (VS), L2.1, VT3.3 (S), VT4.2 (D)
- new net Вих1: R31.1
- new net Вих2: R30.1
- new net Уст.0: R29.1, R31.2
Other:
- note removed: "Вход"
- note removed: "Перегрузка"
- note removed: "Уст. 0"
- note removed: "Уст. тока защиты"
- moved on the sheet: C1, C10, C12, C14, C15, C19, C2, C20, C21, C22, C8, IC2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
